Commit message: Update Etna

File: etna_workcell/urdf/diode_head.xacro (robot description, xacro)
@@ -9,9 +9,5 @@
   <visual>
     <geometry>
-<<<<<<< HEAD
-      <mesh filename="package://etna_workcell/meshes/head_diode/head_diode.stl" />
-=======
       <mesh filename="package://etna_workcell/meshes/head_diode/head.stl" />
->>>>>>> d3ed556e67d821343be06efe0997e8100b6a1ab7
     </geometry>
     <material name="gray">

File: etna_workcell/urdf/etna_workcell.xacro (robot description, xacro)
@@ -52,9 +52,5 @@
   <visual>
     <geometry>
-<<<<<<< HEAD
-      <mesh filename="package://etna_workcell/meshes/cell/cell.stl"/>
-=======
       <mesh filename="package://aimen_workcell/meshes/cell/cell.stl"/>
->>>>>>> d3ed556e67d821343be06efe0997e8100b6a1ab7
     </geometry>
     <origin xyz="0 0 0" />

File: etna_workcell/urdf/fiber_head.xacro (robot description, xacro)
@@ -9,9 +9,5 @@
   <visual>
     <geometry>
-<<<<<<< HEAD
-      <mesh filename="package://etna_workcell/meshes/head/head.stl"/>
-=======
       <mesh filename="package://etna_workcell/meshes/fiber_head/head.stl"/>
->>>>>>> d3ed556e67d821343be06efe0997e8100b6a1ab7
     </geometry>
     <material name="gray">
